Commit message: fixed marco to world and camera config in marco.xacro

File: src/robot_models/marco/marco_description/robots/marco_titanium.urdf.xacro (robot description, xacro)
@@ -29,4 +29,9 @@
   <xacro:include filename="$(find marco_description)/urdf/sensors/usb_cam.urdf.xacro" />
   <!-- Now we can start using the macros included above to define the actual robot -->
+    <link name="world"/>
+    <joint name="world_to_base_footprint" type="fixed">
+        <parent link="world"/>
+        <child link="base_footprint"/>
+    </joint>
   <xacro:base name="base"/>
   <xacro:marco_torso name="torso" parent="base_link"/>
@@ -43,5 +48,5 @@
       <origin xyz="0 0.021 0" rpy="0 0 0" />
       <!-- optical origin -->
-      <origin xyz="0 0 -0.025" rpy="${-90*deg_to_rad} ${90*deg_to_rad} ${-90*deg_to_rad}" />
+      <origin xyz="0 0 0.025" rpy="${0*deg_to_rad} ${-90*deg_to_rad} ${-90*deg_to_rad}" />
   </xacro:usb_cam>
 </robot>
